File: hardware/bench-rev-a/01-inline.kicad_sch (KiCad schematic)
At the start: 16 parts, among them J1 Inline USB-C receptacle; MPN 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, J2 Force A: source / input, J3 Force B: load / output, J4 Kelvin probe pads; NOT force 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, P1 Custom captive USB-C plug

Commit message: Route the firmware bench PCB and record clean native KiCad checks
Parts:
- J1: value Inline USB-C receptacle; MPN open -> USB4115-03-C / USB path 5A MAX; footprint (none) -> PowerWidget:USB_C_Receptacle_GCT_USB4115-03-C
- J2: value Force A: source / input -> 691137710002 / force terminal; footprint (none) -> PowerWidget:Force_5mm_2pin
- J3: value Force B: load / output -> 691137710002 / force terminal; footprint (none) -> PowerWidget:Force_5mm_2pin
- J4: footprint (none) -> PowerWidget:PinHeader_1x04_P2.54mm_Vertical
- P1: value Custom captive USB-C plug -> Captive harness solder termination; footprint (none) -> PowerWidget:Captive_Termination
- R1: footprint (none) -> PowerWidget:WSK2512_5mR
- R2: footprint (none) -> PowerWidget:R_0805_2012Metric
- TP1, TP2, TP3, TP4, TP5, TP6, TP7, TP8, TP9: footprint (none) -> PowerWidget:TestPoint_Pad_D2.0mm
Other:
- moved on the sheet: J2, J3, J4, P1, R1, R2, TP1, TP2, TP3, TP4, TP5, TP6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
