File: hardware/bench-rev-a/02-sensing.kicad_sch (KiCad schematic)
At the start: 17 parts, among them J5 PC I2C / external MCU, J6 INLINE I2C debug, U1 INA228AIDGSR, U2 ISO1641BD

Commit message: Route the firmware bench PCB and record clean native KiCad checks
Parts:
- C1: value 100nF 50V differential -> 100nF 100V differential; footprint (none) -> PowerWidget:C_0805_2012Metric
- C2: value 10nF 63V -> 10nF 100V X7R; footprint (none) -> PowerWidget:C_0805_2012Metric
- C3, C4, C5: footprint (none) -> PowerWidget:C_0805_2012Metric
- J5, J6: footprint (none) -> PowerWidget:PinHeader_1x04_P2.54mm_Vertical
- R3, R4, R5, R6, R7, R8, R9: footprint (none) -> PowerWidget:R_0805_2012Metric
- TP10: footprint (none) -> PowerWidget:TestPoint_Pad_D2.0mm
- U1: footprint Package_SO:VSSOP-10_3x3mm_P0.5mm -> PowerWidget:VSSOP-10_3x3mm_P0.5mm
- U2: footprint Package_SO:SOIC-8_3.9x4.9mm_P1.27mm -> PowerWidget:SOIC-8_3.9x4.9mm_P1.27mm
Other:
- moved on the sheet: C1, C2, C3, C4, C5, J5, J6, R3, R4, R5, R6, R7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
