File: hardware/bench-rev-a/03-supplies.kicad_sch (KiCad schematic)
At the start: 20 parts, among them J7 Floating external 3.3V, U4 TPS7A1601DGNR, U5 TLV75533PDBVR, U7 TPS22919DCKR

Commit message: Route the firmware bench PCB and record clean native KiCad checks
Parts:
- removed R11: 178k 0.1%, symbol Bench:C_R11
- removed R12: 100k 0.1%, symbol Bench:C_R12
- added C20: 22uF 50V X7R MID, PowerWidget:C_1210_3225Metric, symbol Bench:C_C20
- added C21: 22uF 50V X7R MID, PowerWidget:C_1210_3225Metric, symbol Bench:C_C21
- C10, C18, C19, C8, C9: footprint (none) -> PowerWidget:C_0805_2012Metric
- C6: value 1uF 63V effective >=0.1uF -> 1uF 100V X7R; footprint (none) -> PowerWidget:C_1210_3225Metric
- C7: value 4u7 10V effective >=2u2 -> 2u2 10V X7R; footprint (none) -> PowerWidget:C_0805_2012Metric
- J7, JP2, JP3, JP4: footprint (none) -> PowerWidget:PinHeader_1x02_P2.54mm_Vertical
- JP1: footprint (none) -> PowerWidget:PinHeader_1x03_P2.54mm_Vertical
- R10: value 47R 0.25W branch feed -> 10R 0.25W branch feed; footprint (none) -> PowerWidget:R_0805_2012Metric
- R25, R26: footprint (none) -> PowerWidget:R_0805_2012Metric
- U4: value TPS7A1601DGNR -> TPS7A4333DGQR; footprint (none) -> PowerWidget:HVSSOP10_DGQ
- U5: footprint Package_TO_SOT_SMD:SOT-23-5 -> PowerWidget:SOT-23-5
- U7: footprint Package_TO_SOT_SMD:SOT-363_SC-70-6 -> PowerWidget:SOT-363_SC-70-6
Connections:
- net GND_INLINE: now also U4.11 (EP), U4.5 (GND), U4.7 (MVSEL2), C20.2, C21.2; no longer U4.9 (EP)
- net INLINE_LDO_IN: now also U4.10 (IN); no longer U4.5 (EN), U4.8 (IN)
- net INLINE_FB: no longer names the net of U4.2 (NC)
- new net INLINE_MID: C20.1, C21.1, U4.8 (MID_OUT)
- no-connect marks 5 -> 6
Other:
- moved on the sheet: C10, C18, C19, C6, C7, C8, C9, J7, JP1, JP2, JP3, JP4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
