File: hardware/bench-rev-a/04-usb-mcu.kicad_sch (KiCad schematic)
At the start: 17 parts, among them J8 PC reporting USB-C; MPN open, U3 STM32F072CBT6 / 128K flash, U6 USBLC6-2SC6

Commit message: Route the firmware bench PCB and record clean native KiCad checks
Parts:
- C11, C12, C13, C14, C15, C16: footprint (none) -> PowerWidget:C_0805_2012Metric
- J8: value PC reporting USB-C; MPN open -> USB4105-GF-A-120 / reporting; footprint (none) -> PowerWidget:USB_C_Receptacle_GCT_USB4105-xx-A_16P_TopMnt_Horizontal
- R13, R14, R15, R16, R17, R18, R19, R20: footprint (none) -> PowerWidget:R_0805_2012Metric
- U3: footprint Package_QFP:LQFP-48_7x7mm_P0.5mm -> PowerWidget:LQFP-48_7x7mm_P0.5mm
- U6: footprint Package_TO_SOT_SMD:SOT-23-6 -> PowerWidget:SOT-23-6
Connections:
- no-connect marks 29 -> 21
Other:
- note added: "All circuits here are PC domain. No inline USB or CC signal reaches U3. Reporting connector is GCT USB4105."
- note removed: "All circuits here are PC domain. No inline USB or CC signal reaches U3. USB port footprint remains open."
- moved on the sheet: C11, C12, C13, C14, C15, C16, R13, R14, R15, R16, R17, R18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
