File: hardware/bench-rev-a/05-debug.kicad_sch (KiCad schematic)
At the start: 12 parts, among them J10 UART 3.3V logic, J11 Spare GPIO / SPI, J9 Cortex SWD 2x5 1.27mm, SW1 RESET pushbutton, SW2 BOOT pushbutton, SW3 USER pushbutton

Commit message: Route the firmware bench PCB and record clean native KiCad checks
Parts:
- C17: footprint (none) -> PowerWidget:C_0805_2012Metric
- D1: footprint (none) -> PowerWidget:LED_0805_2012Metric
- J10: footprint (none) -> PowerWidget:PinHeader_1x04_P2.54mm_Vertical
- J11: footprint (none) -> PowerWidget:PinHeader_1x08_P2.54mm_Vertical
- J9: footprint (none) -> PowerWidget:PinHeader_2x05_P1.27mm_Vertical
- R21, R22, R23, R24: footprint (none) -> PowerWidget:R_0805_2012Metric
- SW1, SW2, SW3: footprint (none) -> PowerWidget:SW_SPST_TL3342
Other:
- moved on the sheet: C17, D1, J10, J11, R21, R22, R23, R24, SW1, SW2, SW3
